File: IOExpansion/IOExpansion/IOExpansion.sch (KiCad schematic (older format))
At the start: 60 parts, among them J1 Mount_Hole_3.2mm_M3, J10 HEADER 2x20, J11 I2C_5V, J12 I2C_3V3, J13 I2C_ALT_Master, J14 I2C_Debug, J2 Mount_Hole_3.2mm_M3, J3 Mount_Hole_3.2mm_M3, J4 Mount_Hole_3.2mm_M3, J5 UART_5V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

Commit message: Update files for MUTIF09 I/O Expansion Board (Revision 3). Functionality tests were completed on May 21, 2019.
Parts:
- removed C10, C9: 0.1u, Capacitors_THT:C_Disc_D4.3mm_W1.9mm_P5.00mm, symbol C_Small
- removed J7: RTC_SQW, Pin_Headers:Pin_Header_Straight_1x02_Pitch2.54mm, symbol Conn_01x02
- removed JP1: UART Pass-through, Pin_Headers:Pin_Header_Straight_1x02_Pitch2.54mm, symbol Jumper_NO_Small
- removed R3, R4: 1.8K, Resistors_THT:R_Axial_DIN0207_L6.3mm_D2.5mm_P10.16mm_Horizontal, symbol R
- removed U12, U13: PCA9517A, Housings_SOIC:SOIC-8_3.9x4.9mm_Pitch1.27mm, symbol PCA9517A
- removed U5: TXB0104_Breakout, Housings_DIP:DIP-12_W10.16mm, symbol TXB0104_Breakout
- removed U6: PCA9632DP1_Breakout, ioexplib:PCA9632DP1_Breakout, symbol PCA9632DP1_Breakout
- removed U9: PCF8523_Breakout, Pin_Headers:Pin_Header_Straight_1x05_Pitch2.54mm, symbol PCF8523_Breakout
- added C15: 0.1u, Capacitors_THT:C_Disc_D4.3mm_W1.9mm_P5.00mm, symbol C_Small
- added J15: SQW_OUT, Pin_Headers:Pin_Header_Straight_1x05_Pitch2.54mm, symbol Conn_01x05
- added R11, R13: 10K, Resistors_THT:R_Axial_DIN0207_L6.3mm_D2.5mm_P10.16mm_Horizontal, symbol R
- added R14, R15: R, Resistors_THT:R_Axial_DIN0207_L6.3mm_D2.5mm_P10.16mm_Horizontal, symbol R
- added U12: ADuM1250, Housings_DIP:DIP-8_W7.62mm, symbol ADuM1250
- added U5: 4ch_Level_Shifter_BSS138, Housings_DIP:DIP-12_W10.16mm, symbol 4ch_Level_Shifter_BSS138
- added U6: 4ch_Level_Shifter_BSS138(AKI), Housings_DIP:DIP-12_W10.16mm, symbol 4ch_Level_Shifter_BSS138(AKI)
- added U9: DS3231_Breakout, Pin_Headers:Pin_Header_Straight_1x08_Pitch2.54mm, symbol DS3231_Breakout
- J14: value I2C_Debug -> I2C_Debug_3V3
- J9: value SPI _3V3 -> SPI_3V3
- R1, R2: value 1.8K -> 10K
- U10: value PCA9641 -> PCA9641 (or PCA9541)
- U15: footprint TO_SOT_Packages_THT:TO-220-4_Horizontal -> Pin_Headers:Pin_Header_Straight_1x04_Pitch2.54mm
Connections:
- net labels added: AB0, AB1, AB2, AB3, AS0, AS1, AS2, SCL_SLAVE_5V, SDA_SLAVE_5V
- net labels removed: AD0, AD1, AD2, AD3
- wire segments 152 -> 132
- no-connect marks 32 -> 28
Other:
- note added: "16550\nClock Generator"
- note added: "2ch I2C-bus master arbiter"
- note added: "I2C Isolator"
- note added: "I2C-bus to SPI \nbridge"
- note added: "I2C-safe\nLevel shifter"
- note added: "Note: U5 and U6 are mutually exclusive."
- note added: "Optional pull-up resistors"
- note added: "PLD\nAddress decoder\nLogic"
- note added: "RTC (w/ pull-up resistors)"
- note added: "UART to I2C-bus bridge"
- note added: "UART with FIFO"
- moved on the sheet: C8, J12, J13, J14
